File: logi_block/logi_block.kicad_pcb (KiCad board)
At the start: 6 copper layers, 45 x 15 mm, 25 parts, among them J1 Conn_01x02, J2 Conn_02x03_Odd_Even, J3 Conn_02x08_Odd_Even, U1 74HC151, U2 74HC151, U3 74LVC1G157, U4 74LVC1G157, U5 74LVC1G74, U6 74HC164, U7 74HC164

Commit message: Maintenance on schematic Maintenance on PCB (changed serial number for JLCPCB) Added local datasheets Remade pictures Other small refactors...
Parts:
- moved C1 16.6 mm to (120.4, 79.1)
- moved C2 16.6 mm to (120.4, 68.9)
- moved C3 16.6 mm to (115.8, 74.0)
- moved C4 16.6 mm to (104.0, 75.7)
- moved C5 16.6 mm to (104.0, 69.8)
- moved C8 16.6 mm to (87.6, 71.5)
- moved J1 16.6 mm to (122.2, 75.3)
- moved J2 16.6 mm to (87.6, 74.0)
- moved R3 16.6 mm to (100.2, 78.4)
- moved U1 16.6 mm to (109.1, 71.1)
- moved U3 16.6 mm to (117.2, 68.9)
- moved U4 16.6 mm to (117.2, 79.1)
- moved U6 16.6 mm to (98.6, 71.1)
- moved U7 16.6 mm to (98.6, 76.9)
- moved C6 16.6 mm to (94.7, 74.9)
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Other:
- board text added: "2026-06-18"
- board text removed: "2025-09-26"
- board text removed: "JLCJLCJLCJLC"
